File: SndLocket_hw/SndLocket.sch (KiCad schematic (older format))
At the start: 178 parts

Commit message: Proceeding w sch
Parts:
- removed C? (x2): 0.1u, Capacitors:CAP_0603, symbol Tittar_kl:C
- removed Q? (x2): TSOP4856, Sensors:TSOP48xx, symbol Sensors:TSOP48xx
- removed R? (x2): 100R, Resistors:RES_0603, symbol Tittar_kl:R
- added R? (x2): 1k, Resistors:RES_0603, symbol Tittar_kl:R
- added TP? (x2): TESTPOINT, PCB:TESTPOINT_1MM, symbol pcb_details:TESTPOINT
Connections:
- wire segments 696 -> 686
- no-connect marks 29 -> 26
Other:
- note added: "Check if opamp really required"
- note added: "OPAMP2 VINM"
- note added: "OPAMP2 VINP"
- note added: "OPAMP2 VOUT"
- note removed: "CONNECT TO INTERNAL OP AMP"
- moved on the sheet: C?, DA?A, Q?, R?

Commit message: Proceeding
Parts:
- added C? (x2): 18pF, Capacitors:CAP_0603, symbol Tittar_kl:C
- added DD?: CC256x, QFN_DFN:mrQFN76, symbol RF_ICs:CC256x
- added TP? (x5): TESTPOINT, PCB:TESTPOINT_1MM, symbol pcb_details:TESTPOINT
- added XTAL?: 26MHz, Quartz:03225C4, symbol Tittar_kl:CRYSTAL_H
- BLN?: symbol RFICs:BALUN868JOHANSON -> RF_ICs:BALUN868JOHANSON
- DD?: symbol RFICs:CC1101 -> RF_ICs:CC1101
Connections:
- net labels added: HSI_AU_CLK, HSI_AU_FSYNC, HSI_AU_IN, HSI_AU_OUT, MCU_CTS_HSI_RTS, MCU_RTS_HSI_CTS, MCU_RX_HSI_TX, MCU_TX_HSI_RX
- wire segments 686 -> 708
- no-connect marks 26 -> 21
Other:
- moved on the sheet: C?, DD?, L?, Q?, R?, TP?, XL?, XTAL?

Commit message: Proceeding
Parts:
- added TP? (x5): TESTPOINT, PCB:TESTPOINT_1MM, symbol pcb_details:TESTPOINT
Connections:
- net labels added: 32KHZ_1V8, 32KHZ_3V3, AU_CLK_1V8, AU_CLK_3V3, AU_FSYNC_1V8, AU_FSYNC_3V3, AU_IN_1V8, AU_IN_3V3, AU_OUT_1V8, AU_OUT_3V3, MCU_CTS_HSI_RTS_1V8, MCU_CTS_HSI_RTS_3V3, MCU_RTS_HSI_CTS_1V8, MCU_RTS_HSI_CTS_3V3, MCU_RX_HSI_TX_1V8, MCU_RX_HSI_TX_3V3, MCU_TX_HSI_RX_1V8, MCU_TX_HSI_RX_3V3, nSHUTD_1V8, nSHUTD_3V3
- net labels removed: HSI_AU_CLK, HSI_AU_FSYNC, HSI_AU_IN, HSI_AU_OUT, MCU_CTS_HSI_RTS, MCU_RTS_HSI_CTS, MCU_RX_HSI_TX, MCU_TX_HSI_RX
- wire segments 708 -> 726
- no-connect marks 21 -> 22
Other:
- note added: "Hi->Lo"
- note added: "Hi<-Lo"
- moved on the sheet: C?, DD?, TP?, XTAL?

Commit message: .
Other:
- note added: "Hi->Lo 5"
- note added: "Hi<-Lo 5"
Changed lines of the file:
@@
 	1    0    0    -1
 $EndComp
-Text Label 12450 7050 2    50   ~ 0
+Text Label 12650 7150 2    50   ~ 0
 AU_OUT_1V8
-Text Label 12450 6950 2    50   ~ 0
+Text Label 12650 7050 2    50   ~ 0
 AU_IN_1V8
-Text Label 12450 6850 2    50   ~ 0
+Text Label 12650 6950 2    50   ~ 0
 AU_CLK_1V8
-Text Label 12450 6750 2    50   ~ 0
+Text Label 12650 6850 2    50   ~ 0
 AU_FSYNC_1V8
 Text Label 10650 7150 0    50   ~ 0
@@
 Text Notes 10200 7650 2    50   ~ 0
 Hi->Lo
+Text Notes 10200 5550 2    50   ~ 0
+Hi->Lo 5
+Text Notes 10200 5650 2    50   ~ 0
+Hi<-Lo 5
 Wire Bus Line
 	12400 13450 12400 14550

Commit message: Sound routing done
Parts:
- removed R? (x2): 10k, Resistors:RES_0603, symbol Tittar_kl:R
- removed TP? (x8): TESTPOINT, PCB:TESTPOINT_1MM, symbol pcb_details:TESTPOINT
- added C? (x2): 0.1u, Capacitors:CAP_0603, symbol Tittar_kl:C
- added DD? (x14): SN74LVC07, SO_DIL_TSSOP:SO14, symbol standard_logic:6xBufferOD
- added Q?: IRLML6401, SOT:SOT23-3, symbol Transistors_kl:P_3PIN
- added R? (x10): 10k, Resistors:RES_0603, symbol Tittar_kl:R
- added R?: 100k, Resistors:RES_0603, symbol Tittar_kl:R
- added R? (x8): 1k, Resistors:RES_0603, symbol Tittar_kl:R
- added TP? (x8): TESTPOINT, PCB:TESTPOINT_1MM, symbol pcb_details:TESTPOINT
Connections:
- net labels added: +1v8
- wire segments 726 -> 787
- no-connect marks 22 -> 24
Other:
- note added: "AUDIO"
- note added: "CHECK IF 1k REQUIRED"
- note added: "CLK & EN"
- note added: "UART"
- note removed: "Hi->Lo"
- note removed: "Hi->Lo 5"
- note removed: "Hi<-Lo"
- note removed: "Hi<-Lo 5"
- moved on the sheet: C?, DA?, DD?, L?, MIC?, Q?, R?, SW?, TP?, XL?, XTAL?

Commit message: no message
Parts:
- removed C? (x2): 470u, Capacitors:CAP_D, symbol Tittar_kl:CP
- removed Q?: IRLML6401, SOT:SOT23-3, symbol Transistors_kl:P_3PIN
- removed R?: 100k, Resistors:RES_0603, symbol Tittar_kl:R
- removed TP? (x5): TESTPOINT, PCB:TESTPOINT_1MM, symbol pcb_details:TESTPOINT
- added ANT1: ANT_GENERAL, symbol Antennas_kl:ANT_GENERAL
- added C13, C26, C31, C4, C50, C57, C61, C63, C87, C93: 1u, Capacitors:CAP_0603, symbol Tittar_kl:C
- added C40, C46, C47, C48, C51, C54, C55, C58, C62, C64: 0.1u, Capacitors:CAP_0603, symbol Tittar_kl:C
- added C45: 22pF, Capacitors:CAP_0603, symbol Tittar_kl:C
- added C84: 100u, Capacitors:CAP_1206, symbol Tittar_kl:C
- added DA1, DA4: AP7331, SOT:SOT23-5, symbol Power_kl:AP7331
- added DA7: MCP1700, SOT:SOT23-3A, symbol Power_kl:MCP1700
- added FLT1: LFB212G45SG8C341, Radio:FLT_LFB21, symbol RF_ICs:FILTER
- added L1: BLM15, Inductors:IND_0402, symbol Tittar_kl:L
- added Q2: IRLML6401, SOT:SOT23-3, symbol Transistors_kl:P_3PIN
- added R10: 56k, Resistors:RES_0603, symbol Tittar_kl:R
- added R13, R18, R2: 100k, Resistors:RES_0603, symbol Tittar_kl:R
- added R19: 330k, Resistors:RES_0603, symbol Tittar_kl:R
- added R20: 47k, Resistors:RES_0603, symbol Tittar_kl:R
- added R9: 200k, Resistors:RES_0603, symbol Tittar_kl:R
- gave numbers to parts that had none: 202
Connections:
- net labels added: ALO, BT_PWR, BT_PWR_EN, CLO, DCLO, DIG_LDO_OUT, MLDO_OUT, NFC_PWR_EN, SLO
- net labels removed: AU_LRCK, AU_SCLK, AU_SDIN, AU_SDOUT, LED_B, LED_G, LED_R
- wire segments 787 -> 966
- no-connect marks 24 -> 27
Other:
- note added: "Bluetooth: 4v8 + 1v8, up to 115mA"
- note added: "Freqs:\n\nMCU: 12MHz (48 for USB)\nBluetooth: 26MHz\nNFC: 27.12MHz\nAudioCodec: 12MHz from MCU\nRadio: 27MHz"
- note added: "MCU & CC power"
- note added: "Power\n\nMCU: 3v3\nBluetooth: 1v8\nNFC: 3v3\nAudio: 3v3 + Battery\nRadio: 3v3"
- note added: "PullUp when off"
- note removed: "DMA\n\nDMA1 CH2: USART3_TX\nDMA1 CH3: USART3_RX\nDMA1 CH4: USART1TX\nDMA1 CH5: USART1 RX\nDMA1 CH6: USART2RX\nDMA1 CH7: USART2 TX\n\nDMA2 CH1: SPI3 RX\nDMA2 CH2: SPI3 TX\nDMA2 CH3: SPI1 RX\nDMA2 CH4: SPI1 TX\nDMA2 CH5: SDMMC\nDMA2 CH6: SAI1A\nDMA2 CH7: SAI1B"
- note removed: "EXTI IRQs\n\nNFC: PD0\nPMIC: PA2 (WKUP4)\nWIFI_READ: PA3\nBLE_RDYN: PC5 (WKUP5)"
- note removed: "MCU power"
- note removed: "Periphery\n\ni2c1: Sound\ni2c2: AccGyro\nMCO: 12MHz sound\nSAI1: Sound\nSDIO\nSPI1: WiFI\nSPI2: BLE\nSPI3: NFC\nTIM4 C1,C2,C3,C4: LEDs\nTIM5: SysClk\nUSART1: debug\nUSART2: WiFi UART0\nUSART3: WiFi UART2\nUSB\nWKUP1: buttons & ACG\nWKUP2: Power switch\nWKUP4: PMIC\nWKUP5: BLE"
- note removed: "Power\n\nMCU runs @ 48MHz\nIsupp <7mA"
- moved on the sheet: B1, C10, C14, C18, C23, C24, C29, C30, C65, C67, C68, C69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

Commit message: .
Parts:
- removed R31, R32: 0R, Resistors:RES_0603, symbol Tittar_kl:R
- removed TP11, TP12, TP13, TP14, TP3, TP4, TP5, TP6, TP7, TP8: TESTPOINT, PCB:TESTPOINT_1MM, symbol pcb_details:TESTPOINT
- ANT1: footprint (none) -> Antennas:LcktSnd_2d41
- ANT2: footprint Antennas:Locket5 -> Antennas:LcktSnd_868; symbol Antennas_kl:ANT_PCB_MONO_2PIN -> Antennas_kl:ANT_PCB_MONO
- C11, C12, C15, C19, C25, C3, C33, C37, C40, C41, C42, C45, C46, C47, C48, C49, C51, C54, C55, C56, C58, C6, C62, C64, C65, C72, C73, C74, C76, C77, C79, C8, C80, C81, C82, C88, C89, C9, C90, C91: footprint Capacitors:CAP_0603 -> Capacitors:CAP_0402
- C66: value 100pF -> 0.1u; Price 0.5 -> (none); SolderPoints 2 -> (none)
- DA5: footprint QFN_DFN:QFN-32_EP_5x5_Pitch0.5mm -> QFN_DFN:QFN32_EP_5x5_Pitch0.5mm
- DA6: footprint (none) -> SO_DIL_TSSOP:SO8_150MIL
- L2: value Choke -> BLM15
- XL4: footprint Installation:MICROSD_CAP_FIX05A -> Installation:MICROSD_EJECTOR_TFWF1
Connections:
- net ANT1: now also BLN1.1 (Unbal); no longer C66.1
- net GND: now also C66.2; no longer ANT2.2
- net NFC_ANT: now also C43.1, C44.1, C52.1, C53.2, C59.1, C60.2
- net SNS_PWR: now also C66.1
- removed net RF3: BLN1.1 (Unbal), C66.2
Other:
- moved on the sheet: C75, C78, L6
